File: Hardware/PicoWAN.sch (KiCad schematic (older format))
At the start: 45 parts, among them J1 Battery, U1 RFM95W-868S2, U3 MCP73831-2-OT

Commit message: add feather format
Parts:
- added J3: Conn_left, Connector_PinHeader_2.54mm:PinHeader_1x16_P2.54mm_Vertical, symbol Connector:Screw_Terminal_01x16
- added J4: Conn_right, Connector_PinHeader_2.54mm:PinHeader_1x12_P2.54mm_Vertical, symbol Connector:Screw_Terminal_01x12
- U?: symbol MCU_RaspberryPi_and_Boards:RP2040 -> PicoWAN-rescue:RP2040-MCU_RaspberryPi_and_Boards
Connections:
- net labels added: A4, A5, AREF, EN, MISO, MOSI, SCK
- wire segments 199 -> 231
Other:
- note added: "FEATHER PINS"
- moved on the sheet: AE1, C1, C2, C3, C6, C8, C?, D2, D3, D?, J1, P?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

Commit message: add caps and added new pins
Parts:
- added C19: 0.1uF, symbol Device:C_Small
- added R3: 10K, symbol Device:R_Small
- U2: renamed from U?; symbol PicoWAN-rescue:RP2040-MCU_RaspberryPi_and_Boards -> PicoWAN-rescue:RP2040-MCU_RaspberryPi_and_Boards-PicoWAN-rescue
- gave numbers to parts that had none: 30
- renumbered C3 to C16, C6 to C17, C1 to C18, C2 to C5, D2 to D1, D3 to D2, R5 to R6, U1 to U5
Connections:
- net labels added: D24, D25
- net labels removed: A4, A5, AREF, MISO, MOSI, RFM_RST, SCK
- wire segments 231 -> 238
Other:
- moved on the sheet: C18

Commit message: init select footprints
Parts:
- AE1: footprint (none) -> Jumper:SolderJumper-2_P1.3mm_Bridged2Bar_Pad1.0x1.5mm
- C1, C10, C11, C12, C13, C14, C15, C18, C19, C2, C3, C4, C6, C7, C9: footprint (none) -> Capacitor_SMD:C_0805_2012Metric
- C16, C17, C5, C8: footprint Capacitor_SMD:C_0603_1608Metric_Pad1.05x0.95mm_HandSolder -> Capacitor_SMD:C_0805_2012Metric
- D2: footprint LED_SMD:LED_0805_2012Metric_Pad1.15x1.40mm_HandSolder -> LED_SMD:LED_0805_2012Metric
- D3: footprint (none) -> LED_SMD:LED_0805_2012Metric
- R1, R6, R7: footprint Resistor_SMD:R_0603_1608Metric_Pad1.05x0.95mm_HandSolder -> Resistor_SMD:R_0805_2012Metric
- R10, R11, R12, R2, R3, R4, R5, R8, R9: footprint (none) -> Resistor_SMD:R_0805_2012Metric
- U2: footprint RP2040_minimal:RP2040-QFN-56 -> Package_DFN_QFN:QFN-56-1EP_7x7mm_P0.4mm_EP5.6x5.6mm_ThermalVias
- U5: footprint (none) -> RF_Module:HOPERF_RFM9XW_SMD
Changed lines of the file:
@@
 F 0 "C1" V 1111 3595 50  0000 C CNN
 F 1 "22pF" V 1202 3595 50  0000 C CNN
-F 2 "" H 1340 3595 50  0001 C CNN
+F 2 "Capacitor_SMD:C_0805_2012Metric" H 1340 3595 50  0001 C CNN
 F 3 "~" H 1340 3595 50  0001 C CNN
 	1    1340 3595
@@
 F 0 "C2" V 1460 3795 50  0000 C CNN
 F 1 "22pF" V 1530 3795 50  0000 C CNN
-F 2 "" H 1340 3795 50  0001 C CNN
+F 2 "Capacitor_SMD:C_0805_2012Metric" H 1340 3795 50  0001 C CNN
 F 3 "~" H 1340 3795 50  0001 C CNN
 	1    1340 3795
@@
 F 0 "R2" V 1830 3795 50  0000 C CNN
 F 1 "1K" V 1970 3795 50  0000 C CNN
-F 2 "" H 1900 3795 50  0001 C CNN
+F 2 "Resistor_SMD:R_0805_2012Metric" H 1900 3795 50  0001 C CNN
 F 3 "~" H 1900 3795 50  0001 C CNN
 	1    1900 3795
@@
 F 0 "C3" H 1572 6441 50  0000 L CNN
 F 1 "1uF" H 1572 6350 50  0000 L CNN
-F 2 "" H 1480 6395 50  0001 C CNN
+F 2 "Capacitor_SMD:C_0805_2012Metric" H 1480 6395 50  0001 C CNN
 F 3 "~" H 1480 6395 50  0001 C CNN
 	1    1480 6395
@@
 F 0 "C4" H 1892 6441 50  0000 L CNN
 F 1 "0.1uF" H 1830 6325 50  0000 L CNN
-F 2 "" H 1800 6395 50  0001 C CNN
+F 2 "Capacitor_SMD:C_0805_2012Metric" H 1800 6395 50  0001 C CNN
 F 3 "~" H 1800 6395 50  0001 C CNN
 	1    1800 6395
@@
 F 0 "C6" H 2172 6441 50  0000 L CNN
 F 1 "0.1uF" H 2172 6350 50  0000 L CNN
-F 2 "" H 2080 6395 50  0001 C CNN
+F 2 "Capacitor_SMD:C_0805_2012Metric" H 2080 6395 50  0001 C CNN
 F 3 "~" H 2080 6395 50  0001 C CNN
 	1    2080 6395
@@
 F 0 "C7" H 2862 6451 50  0000 L CNN
 F 1 "1uF" H 2862 6360 50  0000 L CNN
-F 2 "" H 2770 6405 50  0001 C CNN
+F 2 "Capacitor_SMD:C_0805_2012Metric" H 2770 6405 50  0001 C CNN
 F 3 "~" H 2770 6405 50  0001 C CNN
 	1    2770 6405
@@
 F 0 "C9" H 3162 6451 50  0000 L CNN
 F 1 "0.1uF" H 3110 6335 50  0000 L CNN
-F 2 "" H 3070 6405 50  0001 C CNN
+F 2 "Capacitor_SMD:C_0805_2012Metric" H 3070 6405 50  0001 C CNN
 F 3 "~" H 3070 6405 50  0001 C CNN
 	1    3070 6405
@@
 F 0 "C10" H 3452 6451 50  0000 L CNN
 F 1 "0.1uF" H 3390 6335 50  0000 L CNN
-F 2 "" H 3360 6405 50  0001 C CNN
+F 2 "Capacitor_SMD:C_0805_2012Metric" H 3360 6405 50  0001 C CNN
 F 3 "~" H 3360 6405 50  0001 C CNN
 	1    3360 6405
@@
 F 0 "C11" H 3752 6451 50  0000 L CNN
 F 1 "0.1uF" H 3700 6335 50  0000 L CNN
-F 2 "" H 3660 6405 50  0001 C CNN
+F 2 "Capacitor_SMD:C_0805_2012Metric" H 3660 6405 50  0001 C CNN
 F 3 "~" H 3660 6405 50  0001 C CNN
 	1    3660 6405
@@
 F 0 "C12" H 4052 6451 50  0000 L CNN
 F 1 "0.1uF" H 4010 6345 50  0000 L CNN
-F 2 "" H 3960 6405 50  0001 C CNN
+F 2 "Capacitor_SMD:C_0805_2012Metric" H 3960 6405 50  0001 C CNN
 F 3 "~" H 3960 6405 50  0001 C CNN
 	1    3960 6405
@@
 F 0 "C13" H 4362 6451 50  0000 L CNN
 F 1 "0.1uF" H 4320 6345 50  0000 L CNN
-F 2 "" H 4270 6405 50  0001 C CNN
+F 2 "Capacitor_SMD:C_0805_2012Metric" H 4270 6405 50  0001 C CNN
 F 3 "~" H 4270 6405 50  0001 C CNN
 	1    4270 6405
@@
 F 0 "C14" H 4662 6451 50  0000 L CNN
 F 1 "0.1uF" H 4610 6335 50  0000 L CNN
-F 2 "" H 4570 6405 50  0001 C CNN
+F 2 "Capacitor_SMD:C_0805_2012Metric" H 4570 6405 50  0001 C CNN
 F 3 "~" H 4570 6405 50  0001 C CNN
 	1    4570 6405
@@
 F 0 "C15" H 4962 6441 50  0000 L CNN
 F 1 "0.1uF" H 4920 6325 50  0000 L CNN
-F 2 "" H 4870 6395 50  0001 C CNN
+F 2 "Capacitor_SMD:C_0805_2012Metric" H 4870 6395 50  0001 C CNN
 F 3 "~" H 4870 6395 50  0001 C CNN
 	1    4870 6395
@@
 F 0 "R8" H 6870 1550 50  0000 L CNN
 F 1 "10K" H 6820 1620 50  0000 L CNN
-F 2 "" H 7010 1600 50  0001 C CNN
+F 2 "Resistor_SMD:R_0805_2012Metric" H 7010 1600 50  0001 C CNN
 F 3 "~" H 7010 1600 50  0001 C CNN
 	1    7010 1600
@@
 F 0 "R11" V 12430 7800 50  0000 C CNN
 F 1 "5K1" V 12500 7810 50  0000 C CNN
-F 2 "" H 12500 7810 50  0001 C CNN
+F 2 "Resistor_SMD:R_0805_2012Metric" H 12500 7810 50  0001 C CNN
 F 3 "~" H 12500 7810 50  0001 C CNN
 	1    12500 7810
@@
 F 0 "R12" V 12570 7920 50  0000 C CNN
 F 1 "5K1" V 12500 7910 50  0000 C CNN
-F 2 "" H 12500 7910 50  0001 C CNN
+F 2 "Resistor_SMD:R_0805_2012Metric" H 12500 7910 50  0001 C CNN
 F 3 "~" H 12500 7910 50  0001 C CNN
 	1    12500 7910
@@
 F 0 "R4" V 4680 1805 50  0000 C CNN
 F 1 "27" V 4750 1805 50  0000 C CNN
-F 2 "" H 4750 1795 50  0001 C CNN
+F 2 "Resistor_SMD:R_0805_2012Metric" H 4750 1795 50  0001 C CNN
 F 3 "~" H 4750 1795 50  0001 C CNN
 	1    4750 1795
@@
 F 0 "R5" V 4830 1895 50  0000 C CNN
 F 1 "27" V 4750 1895 50  0000 C CNN
-F 2 "" H 4750 1895 50  0001 C CNN
+F 2 "Resistor_SMD:R_0805_2012Metric" H 4750 1895 50  0001 C CNN
 F 3 "~" H 4750 1895 50  0001 C CNN
 	1    4750 1895
@@
 F 0 "U2" H 2240 5465 50  0000 C CNN
 F 1 "RP2040" H 4290 1515 50  0000 C CNN
-F 2 "RP2040_minimal:RP2040-QFN-56" H 2550 3495 50  0001 C CNN
+F 2 "Package_DFN_QFN:QFN-56-1EP_7x7mm_P0.4mm_EP5.6x5.6mm_ThermalVias" H 2550 3495 50  0001 C CNN
 F 3 "" H 2550 3495 50  0001 C CNN
 	1    3300 3495
@@
 F 0 "U5" H 8420 9185 50  0000 C CNN
 F 1 "RFM95W-868S2" H 8405 9085 50  0000 C CNN
-F 2 "" H 5520 10275 50  0001 C CNN
+F 2 "RF_Module:HOPERF_RFM9XW_SMD" H 5520 10275 50  0001 C CNN
 F 3 "https://www.hoperf.com/data/upload/portal/20181127/5bfcbea20e9ef.pdf" H 5520 10275 50  0001 C CNN
 	1    8820 8625
@@
 F 0 "C18" H 7602 8546 50  0000 L CNN
 F 1 "0.1uF" H 7602 8455 50  0000 L CNN
-F 2 "" H 7510 8500 50  0001 C CNN
+F 2 "Capacitor_SMD:C_0805_2012Metric" H 7510 8500 50  0001 C CNN
 F 3 "~" H 7510 8500 50  0001 C CNN
 	1    7510 8500
@@
 F 0 "AE1" H 9644 8084 50  0000 L CNN
 F 1 "Antenna_Shield" H 9644 7993 50  0000 L CNN
-F 2 "" H 9500 8145 50  0001 C CNN
+F 2 "Jumper:SolderJumper-2_P1.3mm_Bridged2Bar_Pad1.0x1.5mm" H 9500 8145 50  0001 C CNN
 F 3 "~" H 9500 8145 50  0001 C CNN
 	1    9500 8045
@@
 F 0 "D2" V 6095 9230 50  0000 C CNN
 F 1 "LED" V 6020 9275 50  0000 C CNN
-F 2 "LED_SMD:LED_0805_2012Metric_Pad1.15x1.40mm_HandSolder" H 6000 9140 60  0001 C CNN
+F 2 "LED_SMD:LED_0805_2012Metric" H 6000 9140 60  0001 C CNN
 F 3 "" H 6000 9140 60  0001 C CNN
 F 4 "150080GS75000" H 6000 9140 50  0001 C CNN "manf#"
@@
 F 0 "C16" H 5700 8165 50  0000 L CNN
 F 1 "10uF" H 5700 7965 50  0000 L CNN
-F 2 "Capacitor_SMD:C_0603_1608Metric_Pad1.05x0.95mm_HandSolder" H 5700 8065 60  0001 C CNN
+F 2 "Capacitor_SMD:C_0805_2012Metric" H 5700 8065 60  0001 C CNN
 F 3 "" H 5700 8065 60  0001 C CNN
 F 4 "TCSOM1A106M8R-ZM1" H 5700 8065 50  0001 C CNN "manf#"
@@
 F 0 "C17" H 6350 8740 50  0000 L CNN
 F 1 "10uF" H 6350 8540 50  0000 L CNN
-F 2 "Capacitor_SMD:C_0603_1608Metric_Pad1.05x0.95mm_HandSolder" H 6350 8640 60  0001 C CNN
+F 2 "Capacitor_SMD:C_0805_2012Metric" H 6350 8640 60  0001 C CNN
 F 3 "" H 6350 8640 60  0001 C CNN
 F 4 "TCSOM1A106M8R-ZM1" H 6350 8640 50  0001 C CNN "manf#"
@@
 F 0 "R7" H 6100 8850 40  0000 C CNN
 F 1 "1K" H 6100 8775 40  0000 C CNN
-F 2 "Resistor_SMD:R_0603_1608Metric_Pad1.05x0.95mm_HandSolder" V 5930 8840 30  0001 C CNN
+F 2 "Resistor_SMD:R_0805_2012Metric" V 5930 8840 30  0001 C CNN
 F 3 "" H 6000 8840 60  0001 C CNN
 F 4 "" H 6330 8495 50  0000 C CNN "Place"
@@
 F 0 "R6" H 5080 8895 40  0000 C CNN
 F 1 "2K" H 5110 8820 40  0000 C CNN
-F 2 "Resistor_SMD:R_0603_1608Metric_Pad1.05x0.95mm_HandSolder" V 4910 8885 30  0001 C CNN
+F 2 "Resistor_SMD:R_0805_2012Metric" V 4910 8885 30  0001 C CNN
 F 3 "" H 4980 8885 60  0001 C CNN
 F 4 "" H 5310 8540 50  0000 C CNN "Place"
@@
 F 0 "C5" H 1890 8875 50  0000 L CNN
 F 1 "4.7uF" H 1890 8675 50  0000 L CNN
-F 2 "Capacitor_SMD:C_0603_1608Metric_Pad1.05x0.95mm_HandSolder" H 1890 8775 60  0001 C CNN
+F 2 "Capacitor_SMD:C_0805_2012Metric" H 1890 8775 60  0001 C CNN
 F 3 "" H 1890 8775 60  0001 C CNN
 F 4 "CL10A475KA8NQNC" H 1890 8775 50  0001 C CNN "manf#"
@@
 F 0 "R1" H 1295 8635 40  0000 C CNN
 F 1 "100K" H 1325 8560 40  0000 C CNN
-F 2 "Resistor_SMD:R_0603_1608Metric_Pad1.05x0.95mm_HandSolder" V 1125 8625 30  0001 C CNN
+F 2 "Resistor_SMD:R_0805_2012Metric" V 1125 8625 30  0001 C CNN
 F 3 "" H 1195 8625 60  0001 C CNN
 F 4 "" H 1525 8280 50  0000 C CNN "Place"
@@
 F 0 "C8" H 3090 8845 50  0000 L CNN
 F 1 "1uF" H 3090 8645 50  0000 L CNN
-F 2 "Capacitor_SMD:C_0603_1608Metric_Pad1.05x0.95mm_HandSolder" H 3040 8745 60  0001 C CNN
+F 2 "Capacitor_SMD:C_0805_2012Metric" H 3040 8745 60  0001 C CNN
 F 3 "" H 3040 8745 60  0001 C CNN
 F 4 "CL10A105KA8NNNC" H 3040 8745 50  0001 C CNN "manf#"
@@
 F 0 "R9" V 6959 5365 50  0000 C CNN
 F 1 "1K" V 7050 5365 50  0000 C CNN
-F 2 "" H 7155 5365 50  0001 C CNN
+F 2 "Resistor_SMD:R_0805_2012Metric" H 7155 5365 50  0001 C CNN
 F 3 "~" H 7155 5365 50  0001 C CNN
 	1    7155 5365
@@
 F 0 "D3" H 8748 5965 50  0000 C CNN
 F 1 "LED" H 8748 6056 50  0000 C CNN
-F 2 "" H 8755 6220 50  0001 C CNN
+F 2 "LED_SMD:LED_0805_2012Metric" H 8755 6220 50  0001 C CNN
 F 3 "~" H 8755 6220 50  0001 C CNN
 	1    8755 6220
@@
 F 0 "R10" V 8224 6220 50  0000 C CNN
 F 1 "10K" V 8315 6220 50  0000 C CNN
-F 2 "" H 8420 6220 50  0001 C CNN
+F 2 "Resistor_SMD:R_0805_2012Metric" H 8420 6220 50  0001 C CNN
 F 3 "~" H 8420 6220 50  0001 C CNN
 	1    8420 6220
@@
 F 0 "R3" H 2149 8671 50  0000 L CNN
 F 1 "10K" H 1950 8740 50  0000 L CNN
-F 2 "" H 2090 8625 50  0001 C CNN
+F 2 "Resistor_SMD:R_0805_2012Metric" H 2090 8625 50  0001 C CNN
 F 3 "~" H 2090 8625 50  0001 C CNN
 	1    2090 8625
@@
 F 0 "C19" H 9307 1941 50  0000 L CNN
 F 1 "0.1uF" H 9265 1825 50  0000 L CNN
-F 2 "" H 9215 1895 50  0001 C CNN
+F 2 "Capacitor_SMD:C_0805_2012Metric" H 9215 1895 50  0001 C CNN
 F 3 "~" H 9215 1895 50  0001 C CNN
 	1    9215 1895

Commit message: update to 0603
Parts:
- C1, C10, C11, C12, C13, C14, C15, C16, C17, C18, C19, C2, C3, C4, C5, C6, C7, C8, C9: footprint Capacitor_SMD:C_0805_2012Metric -> Capacitor_SMD:C_0603_1608Metric
- D2, D3: footprint LED_SMD:LED_0805_2012Metric -> LED_SMD:LED_0201_0603Metric
- R1, R10, R11, R12, R2, R3, R4, R5, R6, R7, R8, R9: footprint Resistor_SMD:R_0805_2012Metric -> Resistor_SMD:R_0603_1608Metric
Changed lines of the file:
@@
 F 0 "C1" V 1111 3595 50  0000 C CNN
 F 1 "22pF" V 1202 3595 50  0000 C CNN
-F 2 "Capacitor_SMD:C_0805_2012Metric" H 1340 3595 50  0001 C CNN
+F 2 "Capacitor_SMD:C_0603_1608Metric" H 1340 3595 50  0001 C CNN
 F 3 "~" H 1340 3595 50  0001 C CNN
 	1    1340 3595
@@
 F 0 "C2" V 1460 3795 50  0000 C CNN
 F 1 "22pF" V 1530 3795 50  0000 C CNN
-F 2 "Capacitor_SMD:C_0805_2012Metric" H 1340 3795 50  0001 C CNN
+F 2 "Capacitor_SMD:C_0603_1608Metric" H 1340 3795 50  0001 C CNN
 F 3 "~" H 1340 3795 50  0001 C CNN
 	1    1340 3795
@@
 F 0 "R2" V 1830 3795 50  0000 C CNN
 F 1 "1K" V 1970 3795 50  0000 C CNN
-F 2 "Resistor_SMD:R_0805_2012Metric" H 1900 3795 50  0001 C CNN
+F 2 "Resistor_SMD:R_0603_1608Metric" H 1900 3795 50  0001 C CNN
 F 3 "~" H 1900 3795 50  0001 C CNN
 	1    1900 3795
@@
 F 0 "C3" H 1572 6441 50  0000 L CNN
 F 1 "1uF" H 1572 6350 50  0000 L CNN
-F 2 "Capacitor_SMD:C_0805_2012Metric" H 1480 6395 50  0001 C CNN
+F 2 "Capacitor_SMD:C_0603_1608Metric" H 1480 6395 50  0001 C CNN
 F 3 "~" H 1480 6395 50  0001 C CNN
 	1    1480 6395
@@
 F 0 "C4" H 1892 6441 50  0000 L CNN
 F 1 "0.1uF" H 1830 6325 50  0000 L CNN
-F 2 "Capacitor_SMD:C_0805_2012Metric" H 1800 6395 50  0001 C CNN
+F 2 "Capacitor_SMD:C_0603_1608Metric" H 1800 6395 50  0001 C CNN
 F 3 "~" H 1800 6395 50  0001 C CNN
 	1    1800 6395
@@
 F 0 "C6" H 2172 6441 50  0000 L CNN
 F 1 "0.1uF" H 2172 6350 50  0000 L CNN
-F 2 "Capacitor_SMD:C_0805_2012Metric" H 2080 6395 50  0001 C CNN
+F 2 "Capacitor_SMD:C_0603_1608Metric" H 2080 6395 50  0001 C CNN
 F 3 "~" H 2080 6395 50  0001 C CNN
 	1    2080 6395
@@
 F 0 "C7" H 2862 6451 50  0000 L CNN
 F 1 "1uF" H 2862 6360 50  0000 L CNN
-F 2 "Capacitor_SMD:C_0805_2012Metric" H 2770 6405 50  0001 C CNN
+F 2 "Capacitor_SMD:C_0603_1608Metric" H 2770 6405 50  0001 C CNN
 F 3 "~" H 2770 6405 50  0001 C CNN
 	1    2770 6405
@@
 F 0 "C9" H 3162 6451 50  0000 L CNN
 F 1 "0.1uF" H 3110 6335 50  0000 L CNN
-F 2 "Capacitor_SMD:C_0805_2012Metric" H 3070 6405 50  0001 C CNN
+F 2 "Capacitor_SMD:C_0603_1608Metric" H 3070 6405 50  0001 C CNN
 F 3 "~" H 3070 6405 50  0001 C CNN
 	1    3070 6405
@@
 F 0 "C10" H 3452 6451 50  0000 L CNN
 F 1 "0.1uF" H 3390 6335 50  0000 L CNN
-F 2 "Capacitor_SMD:C_0805_2012Metric" H 3360 6405 50  0001 C CNN
+F 2 "Capacitor_SMD:C_0603_1608Metric" H 3360 6405 50  0001 C CNN
 F 3 "~" H 3360 6405 50  0001 C CNN
 	1    3360 6405
@@
 F 0 "C11" H 3752 6451 50  0000 L CNN
 F 1 "0.1uF" H 3700 6335 50  0000 L CNN
-F 2 "Capacitor_SMD:C_0805_2012Metric" H 3660 6405 50  0001 C CNN
+F 2 "Capacitor_SMD:C_0603_1608Metric" H 3660 6405 50  0001 C CNN
 F 3 "~" H 3660 6405 50  0001 C CNN
 	1    3660 6405
@@
 F 0 "C12" H 4052 6451 50  0000 L CNN
 F 1 "0.1uF" H 4010 6345 50  0000 L CNN
-F 2 "Capacitor_SMD:C_0805_2012Metric" H 3960 6405 50  0001 C CNN
+F 2 "Capacitor_SMD:C_0603_1608Metric" H 3960 6405 50  0001 C CNN
 F 3 "~" H 3960 6405 50  0001 C CNN
 	1    3960 6405
@@
 F 0 "C13" H 4362 6451 50  0000 L CNN
 F 1 "0.1uF" H 4320 6345 50  0000 L CNN
-F 2 "Capacitor_SMD:C_0805_2012Metric" H 4270 6405 50  0001 C CNN
+F 2 "Capacitor_SMD:C_0603_1608Metric" H 4270 6405 50  0001 C CNN
 F 3 "~" H 4270 6405 50  0001 C CNN
 	1    4270 6405
@@
 F 0 "C14" H 4662 6451 50  0000 L CNN
 F 1 "0.1uF" H 4610 6335 50  0000 L CNN
-F 2 "Capacitor_SMD:C_0805_2012Metric" H 4570 6405 50  0001 C CNN
+F 2 "Capacitor_SMD:C_0603_1608Metric" H 4570 6405 50  0001 C CNN
 F 3 "~" H 4570 6405 50  0001 C CNN
 	1    4570 6405
@@
 F 0 "C15" H 4962 6441 50  0000 L CNN
 F 1 "0.1uF" H 4920 6325 50  0000 L CNN
-F 2 "Capacitor_SMD:C_0805_2012Metric" H 4870 6395 50  0001 C CNN
+F 2 "Capacitor_SMD:C_0603_1608Metric" H 4870 6395 50  0001 C CNN
 F 3 "~" H 4870 6395 50  0001 C CNN
 	1    4870 6395
@@
 F 0 "R8" H 6870 1550 50  0000 L CNN
 F 1 "10K" H 6820 1620 50  0000 L CNN
-F 2 "Resistor_SMD:R_0805_2012Metric" H 7010 1600 50  0001 C CNN
+F 2 "Resistor_SMD:R_0603_1608Metric" H 7010 1600 50  0001 C CNN
 F 3 "~" H 7010 1600 50  0001 C CNN
 	1    7010 1600
@@
 F 0 "R11" V 12430 7800 50  0000 C CNN
 F 1 "5K1" V 12500 7810 50  0000 C CNN
-F 2 "Resistor_SMD:R_0805_2012Metric" H 12500 7810 50  0001 C CNN
+F 2 "Resistor_SMD:R_0603_1608Metric" H 12500 7810 50  0001 C CNN
 F 3 "~" H 12500 7810 50  0001 C CNN
 	1    12500 7810
@@
 F 0 "R12" V 12570 7920 50  0000 C CNN
 F 1 "5K1" V 12500 7910 50  0000 C CNN
-F 2 "Resistor_SMD:R_0805_2012Metric" H 12500 7910 50  0001 C CNN
+F 2 "Resistor_SMD:R_0603_1608Metric" H 12500 7910 50  0001 C CNN
 F 3 "~" H 12500 7910 50  0001 C CNN
 	1    12500 7910
@@
 F 0 "R4" V 4680 1805 50  0000 C CNN
 F 1 "27" V 4750 1805 50  0000 C CNN
-F 2 "Resistor_SMD:R_0805_2012Metric" H 4750 1795 50  0001 C CNN
+F 2 "Resistor_SMD:R_0603_1608Metric" H 4750 1795 50  0001 C CNN
 F 3 "~" H 4750 1795 50  0001 C CNN
 	1    4750 1795
@@
 F 0 "R5" V 4830 1895 50  0000 C CNN
 F 1 "27" V 4750 1895 50  0000 C CNN
-F 2 "Resistor_SMD:R_0805_2012Metric" H 4750 1895 50  0001 C CNN
+F 2 "Resistor_SMD:R_0603_1608Metric" H 4750 1895 50  0001 C CNN
 F 3 "~" H 4750 1895 50  0001 C CNN
 	1    4750 1895
@@
 F 0 "C18" H 7602 8546 50  0000 L CNN
 F 1 "0.1uF" H 7602 8455 50  0000 L CNN
-F 2 "Capacitor_SMD:C_0805_2012Metric" H 7510 8500 50  0001 C CNN
+F 2 "Capacitor_SMD:C_0603_1608Metric" H 7510 8500 50  0001 C CNN
 F 3 "~" H 7510 8500 50  0001 C CNN
 	1    7510 8500
@@
 F 0 "D2" V 6095 9230 50  0000 C CNN
 F 1 "LED" V 6020 9275 50  0000 C CNN
-F 2 "LED_SMD:LED_0805_2012Metric" H 6000 9140 60  0001 C CNN
+F 2 "LED_SMD:LED_0201_0603Metric" H 6000 9140 60  0001 C CNN
 F 3 "" H 6000 9140 60  0001 C CNN
 F 4 "150080GS75000" H 6000 9140 50  0001 C CNN "manf#"
@@
 F 0 "C16" H 5700 8165 50  0000 L CNN
 F 1 "10uF" H 5700 7965 50  0000 L CNN
-F 2 "Capacitor_SMD:C_0805_2012Metric" H 5700 8065 60  0001 C CNN
+F 2 "Capacitor_SMD:C_0603_1608Metric" H 5700 8065 60  0001 C CNN
 F 3 "" H 5700 8065 60  0001 C CNN
 F 4 "TCSOM1A106M8R-ZM1" H 5700 8065 50  0001 C CNN "manf#"
@@
 F 0 "C17" H 6350 8740 50  0000 L CNN
 F 1 "10uF" H 6350 8540 50  0000 L CNN
-F 2 "Capacitor_SMD:C_0805_2012Metric" H 6350 8640 60  0001 C CNN
+F 2 "Capacitor_SMD:C_0603_1608Metric" H 6350 8640 60  0001 C CNN
 F 3 "" H 6350 8640 60  0001 C CNN
 F 4 "TCSOM1A106M8R-ZM1" H 6350 8640 50  0001 C CNN "manf#"
@@
 F 0 "R7" H 6100 8850 40  0000 C CNN
 F 1 "1K" H 6100 8775 40  0000 C CNN
-F 2 "Resistor_SMD:R_0805_2012Metric" V 5930 8840 30  0001 C CNN
+F 2 "Resistor_SMD:R_0603_1608Metric" V 5930 8840 30  0001 C CNN
 F 3 "" H 6000 8840 60  0001 C CNN
 F 4 "" H 6330 8495 50  0000 C CNN "Place"
@@
 F 0 "R6" H 5080 8895 40  0000 C CNN
 F 1 "2K" H 5110 8820 40  0000 C CNN
-F 2 "Resistor_SMD:R_0805_2012Metric" V 4910 8885 30  0001 C CNN
+F 2 "Resistor_SMD:R_0603_1608Metric" V 4910 8885 30  0001 C CNN
 F 3 "" H 4980 8885 60  0001 C CNN
 F 4 "" H 5310 8540 50  0000 C CNN "Place"
@@
 F 0 "C5" H 1890 8875 50  0000 L CNN
 F 1 "4.7uF" H 1890 8675 50  0000 L CNN
-F 2 "Capacitor_SMD:C_0805_2012Metric" H 1890 8775 60  0001 C CNN
+F 2 "Capacitor_SMD:C_0603_1608Metric" H 1890 8775 60  0001 C CNN
 F 3 "" H 1890 8775 60  0001 C CNN
 F 4 "CL10A475KA8NQNC" H 1890 8775 50  0001 C CNN "manf#"
@@
 F 0 "R1" H 1295 8635 40  0000 C CNN
 F 1 "100K" H 1325 8560 40  0000 C CNN
-F 2 "Resistor_SMD:R_0805_2012Metric" V 1125 8625 30  0001 C CNN
+F 2 "Resistor_SMD:R_0603_1608Metric" V 1125 8625 30  0001 C CNN
 F 3 "" H 1195 8625 60  0001 C CNN
 F 4 "" H 1525 8280 50  0000 C CNN "Place"
@@
 F 0 "C8" H 3090 8845 50  0000 L CNN
 F 1 "1uF" H 3090 8645 50  0000 L CNN
-F 2 "Capacitor_SMD:C_0805_2012Metric" H 3040 8745 60  0001 C CNN
+F 2 "Capacitor_SMD:C_0603_1608Metric" H 3040 8745 60  0001 C CNN
 F 3 "" H 3040 8745 60  0001 C CNN
 F 4 "CL10A105KA8NNNC" H 3040 8745 50  0001 C CNN "manf#"
@@
 F 0 "R9" V 6959 5365 50  0000 C CNN
 F 1 "1K" V 7050 5365 50  0000 C CNN
-F 2 "Resistor_SMD:R_0805_2012Metric" H 7155 5365 50  0001 C CNN
+F 2 "Resistor_SMD:R_0603_1608Metric" H 7155 5365 50  0001 C CNN
 F 3 "~" H 7155 5365 50  0001 C CNN
 	1    7155 5365
@@
 F 0 "D3" H 8748 5965 50  0000 C CNN
 F 1 "LED" H 8748 6056 50  0000 C CNN
-F 2 "LED_SMD:LED_0805_2012Metric" H 8755 6220 50  0001 C CNN
+F 2 "LED_SMD:LED_0201_0603Metric" H 8755 6220 50  0001 C CNN
 F 3 "~" H 8755 6220 50  0001 C CNN
 	1    8755 6220
@@
 F 0 "R10" V 8224 6220 50  0000 C CNN
 F 1 "10K" V 8315 6220 50  0000 C CNN
-F 2 "Resistor_SMD:R_0805_2012Metric" H 8420 6220 50  0001 C CNN
+F 2 "Resistor_SMD:R_0603_1608Metric" H 8420 6220 50  0001 C CNN
 F 3 "~" H 8420 6220 50  0001 C CNN
 	1    8420 6220
@@
 F 0 "R3" H 2149 8671 50  0000 L CNN
 F 1 "10K" H 1950 8740 50  0000 L CNN
-F 2 "Resistor_SMD:R_0805_2012Metric" H 2090 8625 50  0001 C CNN
+F 2 "Resistor_SMD:R_0603_1608Metric" H 2090 8625 50  0001 C CNN
 F 3 "~" H 2090 8625 50  0001 C CNN
 	1    2090 8625
@@
 F 0 "C19" H 9307 1941 50  0000 L CNN
 F 1 "0.1uF" H 9265 1825 50  0000 L CNN
-F 2 "Capacitor_SMD:C_0805_2012Metric" H 9215 1895 50  0001 C CNN
+F 2 "Capacitor_SMD:C_0603_1608Metric" H 9215 1895 50  0001 C CNN
 F 3 "~" H 9215 1895 50  0001 C CNN
 	1    9215 1895

Commit message: update footprint RP2040
Parts:
- U2: footprint Package_DFN_QFN:QFN-56-1EP_7x7mm_P0.4mm_EP5.6x5.6mm_ThermalVias -> MCU_RaspberryPi_and_Boards:RP2040-QFN-56
Changed lines of the file:
@@
 F 0 "U2" H 2240 5465 50  0000 C CNN
 F 1 "RP2040" H 4290 1515 50  0000 C CNN
-F 2 "Package_DFN_QFN:QFN-56-1EP_7x7mm_P0.4mm_EP5.6x5.6mm_ThermalVias" H 2550 3495 50  0001 C CNN
+F 2 "MCU_RaspberryPi_and_Boards:RP2040-QFN-56" H 2550 3495 50  0001 C CNN
 F 3 "" H 2550 3495 50  0001 C CNN
 	1    3300 3495
