File: Hardware/PicoWAN.sch (KiCad schematic (older format))
At the start: 49 parts, among them J1 Battery, J2 Conn_01x05, J3 Conn_left, J4 Conn_right, P1 USB_C_Plug_USB2.0, Q1 DMG3415U-7, SW1 BOOT, SW2 RESET, U1 AP2112K-3.3, U2 RP2040, U3 MCP73831-2-OT, U4 W25Q32JVZP, U5 RFM95W-868S2, Y1 12Mhz

Commit message: add libraries intialize floor plan
Parts:
- removed J2: Conn_01x05, symbol Connector_Generic:Conn_01x05
- removed Q1: DMG3415U-7, Package_TO_SOT_THT:TO-92L_Inline, symbol Transistor_FET:TP0610L
- added J2: SWD, Connector_PinHeader_2.54mm:PinHeader_1x04_P2.54mm_Vertical, symbol Connector_Generic:Conn_01x04
- added Q1: DMG3415U-7, Package_TO_SOT_SMD:SOT-23, symbol Device:Q_PMOS_GSD
- AE1: footprint Jumper:SolderJumper-2_P1.3mm_Bridged2Bar_Pad1.0x1.5mm -> pico-wan:SMA_EDGE
- D2, D3: footprint LED_SMD:LED_0201_0603Metric -> LED_SMD:LED_0603_1608Metric
- J1: footprint Connector_PinHeader_2.54mm:PinHeader_1x02_P2.54mm_Vertical -> pico-wan:JST_S2B-PH-SM4-TB(LF)(SN)
- SW1, SW2: footprint (none) -> Button_Switch_SMD:SW_SPST_TL3342
- U2: symbol PicoWAN-rescue:RP2040-MCU_RaspberryPi_and_Boards-PicoWAN-rescue -> PicoWAN-rescue:RP2040-MCU_RaspberryPi_and_Boards-PicoWAN-rescue-PicoWAN-rescue
- U4: value W25Q32JVZP -> W25Q16JV; footprint Package_SON:WSON-8-1EP_6x5mm_P1.27mm_EP3.4x4.3mm -> Package_SON:SON-8-1EP_3x2mm_P0.5mm_EP1.4x1.6mm; manf# (none) -> W25Q16JVUXIQ
Connections:
- net labels removed: USB_BOOT
- wire segments 238 -> 237
Changed lines of the file:
@@
 P 7600 1910
 F 0 "U4" H 7330 2270 50  0000 C CNN
-F 1 "W25Q32JVZP" H 7890 2280 50  0000 C CNN
-F 2 "Package_SON:WSON-8-1EP_6x5mm_P1.27mm_EP3.4x4.3mm" H 7600 1910 50  0001 C CNN
+F 1 "W25Q16JV" H 7890 2280 50  0000 C CNN
+F 2 "Package_SON:SON-8-1EP_3x2mm_P0.5mm_EP1.4x1.6mm" H 7600 1910 50  0001 C CNN
 F 3 "http://www.winbond.com/resource-files/w25q32jv%20revg%2003272018%20plus.pdf" H 7600 1910 50  0001 C CNN
+F 4 "W25Q16JVUXIQ" H 7600 1910 50  0001 C CNN "manf#"
 	1    7600 1910
 	1    0    0    -1
@@
 $EndComp
 $Comp
-L Connector_Generic:Conn_01x05 J2
-U 1 1 601DD531
-P 7825 4080
-F 0 "J2" H 7905 4122 50  0000 L CNN
-F 1 "Conn_01x05" H 7905 4031 50  0000 L CNN
-F 2 "" H 7825 4080 50  0001 C CNN
-F 3 "~" H 7825 4080 50  0001 C CNN
-	1    7825 4080
-	1    0    0    -1
-$EndComp
-$Comp
 L Connector:USB_C_Plug_USB2.0 P1
 U 1 1 601DF7B9
@@
 	490  7020 10260 7020
 $Comp
-L PicoWAN-rescue:RP2040-MCU_RaspberryPi_and_Boards-PicoWAN-rescue U2
+L PicoWAN-rescue:RP2040-MCU_RaspberryPi_and_Boards-PicoWAN-rescue-PicoWAN-rescue U2
 U 1 1 6015B581
 P 3300 3495
@@
 F 0 "AE1" H 9644 8084 50  0000 L CNN
 F 1 "Antenna_Shield" H 9644 7993 50  0000 L CNN
-F 2 "Jumper:SolderJumper-2_P1.3mm_Bridged2Bar_Pad1.0x1.5mm" H 9500 8145 50  0001 C CNN
+F 2 "pico-wan:SMA_EDGE" H 9500 8145 50  0001 C CNN
 F 3 "~" H 9500 8145 50  0001 C CNN
 	1    9500 8045
@@
 F 0 "D2" V 6095 9230 50  0000 C CNN
 F 1 "LED" V 6020 9275 50  0000 C CNN
-F 2 "LED_SMD:LED_0201_0603Metric" H 6000 9140 60  0001 C CNN
+F 2 "LED_SMD:LED_0603_1608Metric" H 6000 9140 60  0001 C CNN
 F 3 "" H 6000 9140 60  0001 C CNN
 F 4 "150080GS75000" H 6000 9140 50  0001 C CNN "manf#"
@@
 F 0 "J1" H 4485 8702 50  0000 L CNN
 F 1 "Battery" H 4485 8611 50  0000 L CNN
-F 2 "Connector_PinHeader_2.54mm:PinHeader_1x02_P2.54mm_Vertical" H 4405 8710 50  0001 C CNN
+F 2 "pico-wan:JST_S2B-PH-SM4-TB(LF)(SN)" H 4405 8710 50  0001 C CNN
 F 3 "~" H 4405 8710 50  0001 C CNN
 F 4 "AR0165" H 4405 8710 50  0001 C CNN "manf#"
@@
 L power:+3V3 #PWR018
 U 1 1 5FD18795
-P 3040 8395
-F 0 "#PWR018" H 3040 8495 40  0001 C CNN
-F 1 "+3V3" H 2920 8425 40  0000 C CNN
-F 2 "" H 3040 8395 60  0001 C CNN
-F 3 "" H 3040 8395 60  0001 C CNN
-	1    3040 8395
-	1    0    0    -1
-$EndComp
-Wire Wire Line
-	3040 8395 3040 8425
+P 3040 8255
+F 0 "#PWR018" H 3040 8355 40  0001 C CNN
+F 1 "+3V3" H 3040 8395 40  0000 C CNN
+F 2 "" H 3040 8255 60  0001 C CNN
+F 3 "" H 3040 8255 60  0001 C CNN
+	1    3040 8255
+	1    0    0    -1
+$EndComp
+Wire Wire Line
+	3040 8255 3040 8425
 Wire Wire Line
 	1890 8425 1890 8625
@@
 U 1 1 5FDEAA56
 P 2490 8525
-F 0 "U1" H 2490 8867 50  0000 C CNN
-F 1 "AP2112K-3.3" H 2490 8776 50  0000 C CNN
+F 0 "U1" H 2630 8265 50  0000 C CNN
+F 1 "AP2112K-3.3" H 2530 8760 50  0000 C CNN
 F 2 "Package_TO_SOT_SMD:SOT-23-5" H 2490 8850 50  0001 C CNN
 F 3 "https://www.diodes.com/assets/Datasheets/AP2112.pdf" H 2490 8625 50  0001 C CNN
@@
 F 0 "SW2" H 6730 6500 50  0000 C CNN
 F 1 "RESET" H 6730 6409 50  0000 C CNN
-F 2 "" H 6730 6415 50  0001 C CNN
+F 2 "Button_Switch_SMD:SW_SPST_TL3342" H 6730 6415 50  0001 C CNN
 F 3 "~" H 6730 6415 50  0001 C CNN
 	1    6730 6215
@@
 F 0 "SW1" H 6715 5650 50  0000 C CNN
 F 1 "BOOT" H 6715 5559 50  0000 C CNN
-F 2 "" H 6715 5565 50  0001 C CNN
+F 2 "Button_Switch_SMD:SW_SPST_TL3342" H 6715 5565 50  0001 C CNN
 F 3 "~" H 6715 5565 50  0001 C CNN
 	1    6715 5365
@@
 	0    1    1    0
 $EndComp
-Wire Wire Line
-	7255 5365 7385 5365
-Text Label 7385 5365 0    50   ~ 0
-USB_BOOT
 Text Label 7070 6215 0    50   ~ 0
 RST
@@
 F 0 "D3" H 8748 5965 50  0000 C CNN
 F 1 "LED" H 8748 6056 50  0000 C CNN
-F 2 "LED_SMD:LED_0201_0603Metric" H 8755 6220 50  0001 C CNN
+F 2 "LED_SMD:LED_0603_1608Metric" H 8755 6220 50  0001 C CNN
 F 3 "~" H 8755 6220 50  0001 C CNN
 	1    8755 6220
@@
 Wire Wire Line
 	7625 4080 7520 4080
-Wire Wire Line
-	7625 4280 7510 4280
 Text Label 7505 3980 2    50   ~ 0
 SWDIO
@@
 	1    0    0    -1
 $EndComp
-Text Label 7510 4280 0    50   ~ 0
-RST
 Wire Wire Line
 	7210 4180 7210 4255
@@
 Wire Wire Line
 	4550 2795 4665 2795
-$Comp
-L Transistor_FET:TP0610L Q1
-U 1 1 604B8D73
-P 1685 8145
-F 0 "Q1" H 1889 8191 50  0000 L CNN
-F 1 "DMG3415U-7" H 1830 8295 50  0000 L CNN
-F 2 "Package_TO_SOT_THT:TO-92L_Inline" H 1885 8070 50  0001 L CIN
-F 3 "http://www.vishay.com/docs/70209/70209.pdf" H 1685 8145 50  0001 L CNN
-	1    1685 8145
-	1    0    0    -1
-$EndComp
 Wire Notes Line
 	7140 7040 7140 11135
@@
 	1    0    0    -1
 $EndComp
+Text Label 7580 5365 0    50   ~ 0
+QSPI_CS
+Wire Wire Line
+	7255 5365 7580 5365
+$Comp
+L Connector_Generic:Conn_01x04 J2
+U 1 1 602B8168
+P 7825 3980
+F 0 "J2" H 7905 3972 50  0000 L CNN
+F 1 "SWD" H 7905 3881 50  0000 L CNN
+F 2 "Connector_PinHeader_2.54mm:PinHeader_1x04_P2.54mm_Vertical" H 7825 3980 50  0001 C CNN
+F 3 "~" H 7825 3980 50  0001 C CNN
+	1    7825 3980
+	1    0    0    -1
+$EndComp
+$Comp
+L Device:Q_PMOS_GSD Q1
+U 1 1 6030D332
+P 1685 8145
+F 0 "Q1" H 1889 8191 50  0000 L CNN
+F 1 "DMG3415U-7" H 1889 8100 50  0000 L CNN
+F 2 "Package_TO_SOT_SMD:SOT-23" H 1885 8245 50  0001 C CNN
+F 3 "~" H 1685 8145 50  0001 C CNN
+	1    1685 8145
+	1    0    0    -1
+$EndComp

Commit message: Change_footprint
Parts:
- C10, C11, C12, C13, C14, C15, C16, C17, C18, C19, C3, C4, C5, C6, C7, C8, C9: footprint Capacitor_SMD:C_0603_1608Metric -> Capacitor_SMD:C_0402_1005Metric
- P1: symbol Connector:USB_C_Plug_USB2.0 -> PicoWAN-rescue:USB_C_Plug_USB2.0-Connector
- R10, R3, R4, R5, R7, R8, R9: footprint Resistor_SMD:R_0603_1608Metric -> Resistor_SMD:R_0402_1005Metric
- R2: footprint Resistor_SMD:R_0603_1608Metric -> Resistor_SMD:R_0603_1608Metric_Pad1.05x0.95mm_HandSolder
- U1: symbol Regulator_Linear:AP2112K-3.3 -> PicoWAN-rescue:AP2112K-3.3-Regulator_Linear
- Y1: footprint (none) -> Crystal:Crystal_SMD_2520-4Pin_2.5x2.0mm; manf# (none) -> C709001
Changed lines of the file:
@@
 F 0 "Y1" V 1524 3783 50  0000 L CNN
 F 1 "12Mhz" V 1410 3575 50  0000 L CNN
-F 2 "" H 1570 3695 50  0001 C CNN
-F 3 "~" H 1570 3695 50  0001 C CNN
+F 2 "Crystal:Crystal_SMD_2520-4Pin_2.5x2.0mm" H 1570 3695 50  0001 C CNN
+F 3 "https://lcsc.com/product-detail/SMD-Crystal-Resonators_JWT-CM4012M00020T8188026_C709001.html" H 1570 3695 50  0001 C CNN
+F 4 "C709001" H 1570 3695 50  0001 C CNN "manf#"
 	1    1570 3695
 	0    1    1    0
@@
 F 0 "R2" V 1830 3795 50  0000 C CNN
 F 1 "1K" V 1970 3795 50  0000 C CNN
-F 2 "Resistor_SMD:R_0603_1608Metric" H 1900 3795 50  0001 C CNN
+F 2 "Resistor_SMD:R_0603_1608Metric_Pad1.05x0.95mm_HandSolder" H 1900 3795 50  0001 C CNN
 F 3 "~" H 1900 3795 50  0001 C CNN
 	1    1900 3795
@@
 F 0 "C3" H 1572 6441 50  0000 L CNN
 F 1 "1uF" H 1572 6350 50  0000 L CNN
-F 2 "Capacitor_SMD:C_0603_1608Metric" H 1480 6395 50  0001 C CNN
+F 2 "Capacitor_SMD:C_0402_1005Metric" H 1480 6395 50  0001 C CNN
 F 3 "~" H 1480 6395 50  0001 C CNN
 	1    1480 6395
@@
 F 0 "C4" H 1892 6441 50  0000 L CNN
 F 1 "0.1uF" H 1830 6325 50  0000 L CNN
-F 2 "Capacitor_SMD:C_0603_1608Metric" H 1800 6395 50  0001 C CNN
+F 2 "Capacitor_SMD:C_0402_1005Metric" H 1800 6395 50  0001 C CNN
 F 3 "~" H 1800 6395 50  0001 C CNN
 	1    1800 6395
@@
 F 0 "C6" H 2172 6441 50  0000 L CNN
 F 1 "0.1uF" H 2172 6350 50  0000 L CNN
-F 2 "Capacitor_SMD:C_0603_1608Metric" H 2080 6395 50  0001 C CNN
+F 2 "Capacitor_SMD:C_0402_1005Metric" H 2080 6395 50  0001 C CNN
 F 3 "~" H 2080 6395 50  0001 C CNN
 	1    2080 6395
@@
 F 0 "C7" H 2862 6451 50  0000 L CNN
 F 1 "1uF" H 2862 6360 50  0000 L CNN
-F 2 "Capacitor_SMD:C_0603_1608Metric" H 2770 6405 50  0001 C CNN
+F 2 "Capacitor_SMD:C_0402_1005Metric" H 2770 6405 50  0001 C CNN
 F 3 "~" H 2770 6405 50  0001 C CNN
 	1    2770 6405
@@
 F 0 "C9" H 3162 6451 50  0000 L CNN
 F 1 "0.1uF" H 3110 6335 50  0000 L CNN
-F 2 "Capacitor_SMD:C_0603_1608Metric" H 3070 6405 50  0001 C CNN
+F 2 "Capacitor_SMD:C_0402_1005Metric" H 3070 6405 50  0001 C CNN
 F 3 "~" H 3070 6405 50  0001 C CNN
 	1    3070 6405
@@
 F 0 "C10" H 3452 6451 50  0000 L CNN
 F 1 "0.1uF" H 3390 6335 50  0000 L CNN
-F 2 "Capacitor_SMD:C_0603_1608Metric" H 3360 6405 50  0001 C CNN
+F 2 "Capacitor_SMD:C_0402_1005Metric" H 3360 6405 50  0001 C CNN
 F 3 "~" H 3360 6405 50  0001 C CNN
 	1    3360 6405
@@
 F 0 "C11" H 3752 6451 50  0000 L CNN
 F 1 "0.1uF" H 3700 6335 50  0000 L CNN
-F 2 "Capacitor_SMD:C_0603_1608Metric" H 3660 6405 50  0001 C CNN
+F 2 "Capacitor_SMD:C_0402_1005Metric" H 3660 6405 50  0001 C CNN
 F 3 "~" H 3660 6405 50  0001 C CNN
 	1    3660 6405
@@
 F 0 "C12" H 4052 6451 50  0000 L CNN
 F 1 "0.1uF" H 4010 6345 50  0000 L CNN
-F 2 "Capacitor_SMD:C_0603_1608Metric" H 3960 6405 50  0001 C CNN
+F 2 "Capacitor_SMD:C_0402_1005Metric" H 3960 6405 50  0001 C CNN
 F 3 "~" H 3960 6405 50  0001 C CNN
 	1    3960 6405
@@
 F 0 "C13" H 4362 6451 50  0000 L CNN
 F 1 "0.1uF" H 4320 6345 50  0000 L CNN
-F 2 "Capacitor_SMD:C_0603_1608Metric" H 4270 6405 50  0001 C CNN
+F 2 "Capacitor_SMD:C_0402_1005Metric" H 4270 6405 50  0001 C CNN
 F 3 "~" H 4270 6405 50  0001 C CNN
 	1    4270 6405
@@
 F 0 "C14" H 4662 6451 50  0000 L CNN
 F 1 "0.1uF" H 4610 6335 50  0000 L CNN
-F 2 "Capacitor_SMD:C_0603_1608Metric" H 4570 6405 50  0001 C CNN
+F 2 "Capacitor_SMD:C_0402_1005Metric" H 4570 6405 50  0001 C CNN
 F 3 "~" H 4570 6405 50  0001 C CNN
 	1    4570 6405
@@
 F 0 "C15" H 4962 6441 50  0000 L CNN
 F 1 "0.1uF" H 4920 6325 50  0000 L CNN
-F 2 "Capacitor_SMD:C_0603_1608Metric" H 4870 6395 50  0001 C CNN
+F 2 "Capacitor_SMD:C_0402_1005Metric" H 4870 6395 50  0001 C CNN
 F 3 "~" H 4870 6395 50  0001 C CNN
 	1    4870 6395
@@
 F 0 "R8" H 6870 1550 50  0000 L CNN
 F 1 "10K" H 6820 1620 50  0000 L CNN
-F 2 "Resistor_SMD:R_0603_1608Metric" H 7010 1600 50  0001 C CNN
+F 2 "Resistor_SMD:R_0402_1005Metric" H 7010 1600 50  0001 C CNN
 F 3 "~" H 7010 1600 50  0001 C CNN
 	1    7010 1600
@@
 $EndComp
 $Comp
-L Connector:USB_C_Plug_USB2.0 P1
+L PicoWAN-rescue:USB_C_Plug_USB2.0-Connector P1
 U 1 1 601DF7B9
 P 11740 8210
@@
 F 0 "R4" V 4680 1805 50  0000 C CNN
 F 1 "27" V 4750 1805 50  0000 C CNN
-F 2 "Resistor_SMD:R_0603_1608Metric" H 4750 1795 50  0001 C CNN
+F 2 "Resistor_SMD:R_0402_1005Metric" H 4750 1795 50  0001 C CNN
 F 3 "~" H 4750 1795 50  0001 C CNN
 	1    4750 1795
@@
 F 0 "R5" V 4830 1895 50  0000 C CNN
 F 1 "27" V 4750 1895 50  0000 C CNN
-F 2 "Resistor_SMD:R_0603_1608Metric" H 4750 1895 50  0001 C CNN
+F 2 "Resistor_SMD:R_0402_1005Metric" H 4750 1895 50  0001 C CNN
 F 3 "~" H 4750 1895 50  0001 C CNN
 	1    4750 1895
@@
 F 0 "C18" H 7602 8546 50  0000 L CNN
 F 1 "0.1uF" H 7602 8455 50  0000 L CNN
-F 2 "Capacitor_SMD:C_0603_1608Metric" H 7510 8500 50  0001 C CNN
+F 2 "Capacitor_SMD:C_0402_1005Metric" H 7510 8500 50  0001 C CNN
 F 3 "~" H 7510 8500 50  0001 C CNN
 	1    7510 8500
@@
 F 0 "C16" H 5700 8165 50  0000 L CNN
 F 1 "10uF" H 5700 7965 50  0000 L CNN
-F 2 "Capacitor_SMD:C_0603_1608Metric" H 5700 8065 60  0001 C CNN
+F 2 "Capacitor_SMD:C_0402_1005Metric" H 5700 8065 60  0001 C CNN
 F 3 "" H 5700 8065 60  0001 C CNN
 F 4 "TCSOM1A106M8R-ZM1" H 5700 8065 50  0001 C CNN "manf#"
@@
 F 0 "C17" H 6350 8740 50  0000 L CNN
 F 1 "10uF" H 6350 8540 50  0000 L CNN
-F 2 "Capacitor_SMD:C_0603_1608Metric" H 6350 8640 60  0001 C CNN
+F 2 "Capacitor_SMD:C_0402_1005Metric" H 6350 8640 60  0001 C CNN
 F 3 "" H 6350 8640 60  0001 C CNN
 F 4 "TCSOM1A106M8R-ZM1" H 6350 8640 50  0001 C CNN "manf#"
@@
 F 0 "R7" H 6100 8850 40  0000 C CNN
 F 1 "1K" H 6100 8775 40  0000 C CNN
-F 2 "Resistor_SMD:R_0603_1608Metric" V 5930 8840 30  0001 C CNN
+F 2 "Resistor_SMD:R_0402_1005Metric" V 5930 8840 30  0001 C CNN
 F 3 "" H 6000 8840 60  0001 C CNN
 F 4 "" H 6330 8495 50  0000 C CNN "Place"
@@
 F 0 "C5" H 1890 8875 50  0000 L CNN
 F 1 "4.7uF" H 1890 8675 50  0000 L CNN
-F 2 "Capacitor_SMD:C_0603_1608Metric" H 1890 8775 60  0001 C CNN
+F 2 "Capacitor_SMD:C_0402_1005Metric" H 1890 8775 60  0001 C CNN
 F 3 "" H 1890 8775 60  0001 C CNN
 F 4 "CL10A475KA8NQNC" H 1890 8775 50  0001 C CNN "manf#"
@@
 F 0 "C8" H 3090 8845 50  0000 L CNN
 F 1 "1uF" H 3090 8645 50  0000 L CNN
-F 2 "Capacitor_SMD:C_0603_1608Metric" H 3040 8745 60  0001 C CNN
+F 2 "Capacitor_SMD:C_0402_1005Metric" H 3040 8745 60  0001 C CNN
 F 3 "" H 3040 8745 60  0001 C CNN
 F 4 "CL10A105KA8NNNC" H 3040 8745 50  0001 C CNN "manf#"
@@
 $EndComp
 $Comp
-L Regulator_Linear:AP2112K-3.3 U1
+L PicoWAN-rescue:AP2112K-3.3-Regulator_Linear U1
 U 1 1 5FDEAA56
 P 2490 8525
@@
 F 0 "R9" V 6959 5365 50  0000 C CNN
 F 1 "1K" V 7050 5365 50  0000 C CNN
-F 2 "Resistor_SMD:R_0603_1608Metric" H 7155 5365 50  0001 C CNN
+F 2 "Resistor_SMD:R_0402_1005Metric" H 7155 5365 50  0001 C CNN
 F 3 "~" H 7155 5365 50  0001 C CNN
 	1    7155 5365
@@
 F 0 "R10" V 8224 6220 50  0000 C CNN
 F 1 "10K" V 8315 6220 50  0000 C CNN
-F 2 "Resistor_SMD:R_0603_1608Metric" H 8420 6220 50  0001 C CNN
+F 2 "Resistor_SMD:R_0402_1005Metric" H 8420 6220 50  0001 C CNN
 F 3 "~" H 8420 6220 50  0001 C CNN
 	1    8420 6220
@@
 F 0 "R3" H 2149 8671 50  0000 L CNN
 F 1 "10K" H 1950 8740 50  0000 L CNN
-F 2 "Resistor_SMD:R_0603_1608Metric" H 2090 8625 50  0001 C CNN
+F 2 "Resistor_SMD:R_0402_1005Metric" H 2090 8625 50  0001 C CNN
 F 3 "~" H 2090 8625 50  0001 C CNN
 	1    2090 8625
@@
 F 0 "C19" H 9307 1941 50  0000 L CNN
 F 1 "0.1uF" H 9265 1825 50  0000 L CNN
-F 2 "Capacitor_SMD:C_0603_1608Metric" H 9215 1895 50  0001 C CNN
+F 2 "Capacitor_SMD:C_0402_1005Metric" H 9215 1895 50  0001 C CNN
 F 3 "~" H 9215 1895 50  0001 C CNN
 	1    9215 1895

Commit message: Init_rout
Parts:
- C1, C2: footprint Capacitor_SMD:C_0603_1608Metric -> Capacitor_SMD:C_0402_1005Metric
- R2: footprint Resistor_SMD:R_0603_1608Metric_Pad1.05x0.95mm_HandSolder -> Resistor_SMD:R_0402_1005Metric
Changed lines of the file:
@@
 F 0 "C1" V 1111 3595 50  0000 C CNN
 F 1 "22pF" V 1202 3595 50  0000 C CNN
-F 2 "Capacitor_SMD:C_0603_1608Metric" H 1340 3595 50  0001 C CNN
+F 2 "Capacitor_SMD:C_0402_1005Metric" H 1340 3595 50  0001 C CNN
 F 3 "~" H 1340 3595 50  0001 C CNN
 	1    1340 3595
@@
 F 0 "C2" V 1460 3795 50  0000 C CNN
 F 1 "22pF" V 1530 3795 50  0000 C CNN
-F 2 "Capacitor_SMD:C_0603_1608Metric" H 1340 3795 50  0001 C CNN
+F 2 "Capacitor_SMD:C_0402_1005Metric" H 1340 3795 50  0001 C CNN
 F 3 "~" H 1340 3795 50  0001 C CNN
 	1    1340 3795
@@
 F 0 "R2" V 1830 3795 50  0000 C CNN
 F 1 "1K" V 1970 3795 50  0000 C CNN
-F 2 "Resistor_SMD:R_0603_1608Metric_Pad1.05x0.95mm_HandSolder" H 1900 3795 50  0001 C CNN
+F 2 "Resistor_SMD:R_0402_1005Metric" H 1900 3795 50  0001 C CNN
 F 3 "~" H 1900 3795 50  0001 C CNN
 	1    1900 3795
