File: Hardware/PicoWAN.sch (KiCad schematic (older format))
At the start: 49 parts, among them J1 Battery, J2 SWD, J3 Conn_left, J4 Conn_right, P1 USB_C_Plug_USB2.0, Q1 DMG3415U-7, SW1 BOOT, SW2 RESET, U1 AP2112K-3.3, U2 RP2040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

Commit message: Move_Micro
Parts:
- AE1: footprint pico-wan:SMA_EDGE -> Connectors:MOLEX_1661
Changed lines of the file:
@@
 F 0 "AE1" H 9644 8084 50  0000 L CNN
 F 1 "Antenna_Shield" H 9644 7993 50  0000 L CNN
-F 2 "pico-wan:SMA_EDGE" H 9500 8145 50  0001 C CNN
+F 2 "Connectors:MOLEX_1661" H 9500 8145 50  0001 C CNN
 F 3 "~" H 9500 8145 50  0001 C CNN
 	1    9500 8045

Commit message: Sch
Parts:
- U4: footprint Package_SON:SON-8-1EP_3x2mm_P0.5mm_EP1.4x1.6mm -> hunter-cat-nfc:PSON50P200X300X50-9N
Changed lines of the file:
@@
 F 0 "U4" H 7330 2270 50  0000 C CNN
 F 1 "W25Q16JV" H 7890 2280 50  0000 C CNN
-F 2 "Package_SON:SON-8-1EP_3x2mm_P0.5mm_EP1.4x1.6mm" H 7600 1910 50  0001 C CNN
+F 2 "hunter-cat-nfc:PSON50P200X300X50-9N" H 7600 1910 50  0001 C CNN
 F 3 "http://www.winbond.com/resource-files/w25q32jv%20revg%2003272018%20plus.pdf" H 7600 1910 50  0001 C CNN
 F 4 "W25Q16JVUXIQ" H 7600 1910 50  0001 C CNN "manf#"

Commit message: update crystal and traces
Parts:
- removed Y1: 12Mhz, Crystal:Crystal_SMD_2520-4Pin_2.5x2.0mm, symbol Device:Crystal_Small
- added Y2: 12Mhz, Crystal:Crystal_SMD_2520-4Pin_2.5x2.0mm, symbol Device:Crystal_GND2
- R1, R6, R7: Note not needed since we don't read VCC_SIM -> (none)
Connections:
- net GND: now also Y2.2
- net at C1.1, U2.20 (XIN): now also Y2.1
- net at C2.1, R2.1: now also Y2.3
Other:
- moved on the sheet: C1, C2
Changed lines of the file:
@@
 SWDIO
-$Comp
-L Device:Crystal_Small Y1
-U 1 1 60168897
-P 1570 3695
-F 0 "Y1" V 1524 3783 50  0000 L CNN
-F 1 "12Mhz" V 1410 3575 50  0000 L CNN
-F 2 "Crystal:Crystal_SMD_2520-4Pin_2.5x2.0mm" H 1570 3695 50  0001 C CNN
-F 3 "https://lcsc.com/product-detail/SMD-Crystal-Resonators_JWT-CM4012M00020T8188026_C709001.html" H 1570 3695 50  0001 C CNN
-F 4 "C709001" H 1570 3695 50  0001 C CNN "manf#"
-	1    1570 3695
-	0    1    1    0
-$EndComp
-Wire Wire Line
-	1570 3795 1800 3795
-Wire Wire Line
-	1570 3795 1440 3795
-Connection ~ 1570 3795
-Wire Wire Line
-	1570 3595 1440 3595
-Connection ~ 1570 3595
 $Comp
 L Device:C_Small C1
 U 1 1 6016C552
-P 1340 3595
-F 0 "C1" V 1111 3595 50  0000 C CNN
-F 1 "22pF" V 1202 3595 50  0000 C CNN
-F 2 "Capacitor_SMD:C_0402_1005Metric" H 1340 3595 50  0001 C CNN
-F 3 "~" H 1340 3595 50  0001 C CNN
-	1    1340 3595
-	0    1    1    0
+P 975 4155
+F 0 "C1" V 746 4155 50  0000 C CNN
+F 1 "22pF" V 837 4155 50  0000 C CNN
+F 2 "Capacitor_SMD:C_0402_1005Metric" H 975 4155 50  0001 C CNN
+F 3 "~" H 975 4155 50  0001 C CNN
+	1    975  4155
+	1    0    0    -1
 $EndComp
 $Comp
 L Device:C_Small C2
 U 1 1 6016CD06
-P 1340 3795
-F 0 "C2" V 1460 3795 50  0000 C CNN
-F 1 "22pF" V 1530 3795 50  0000 C CNN
-F 2 "Capacitor_SMD:C_0402_1005Metric" H 1340 3795 50  0001 C CNN
-F 3 "~" H 1340 3795 50  0001 C CNN
-	1    1340 3795
-	0    1    1    0
-$EndComp
-Wire Wire Line
-	1240 3595 1180 3595
-Wire Wire Line
-	1180 3595 1180 3705
-Wire Wire Line
-	1180 3795 1240 3795
-Wire Wire Line
-	1180 3705 1090 3705
-Connection ~ 1180 3705
-Wire Wire Line
-	1180 3705 1180 3795
-$Comp
-L power:GND #PWR01
-U 1 1 6016E9D0
-P 1090 3705
-F 0 "#PWR01" H 1090 3455 50  0001 C CNN
-F 1 "GND" H 1095 3532 50  0000 C CNN
-F 2 "" H 1090 3705 50  0001 C CNN
-F 3 "" H 1090 3705 50  0001 C CNN
-	1    1090 3705
+P 1475 4180
+F 0 "C2" V 1595 4180 50  0000 C CNN
+F 1 "22pF" V 1665 4180 50  0000 C CNN
+F 2 "Capacitor_SMD:C_0402_1005Metric" H 1475 4180 50  0001 C CNN
+F 3 "~" H 1475 4180 50  0001 C CNN
+	1    1475 4180
 	1    0    0    -1
 $EndComp
@@
 Wire Wire Line
 	4550 2495 4660 2495
-Text Label 4660 2195 0    50   ~ 0
-TX
-Text Label 4660 2295 0    50   ~ 0
-RX
 Text Label 4650 2395 0    50   ~ 0
 SDA
@@
 	2050 3795 2000 3795
 Wire Wire Line
-	1570 3595 2050 3595
-Wire Wire Line
 	4550 4895 4650 4895
 Wire Wire Line
@@
 F 3 "" H 6000 8840 60  0001 C CNN
 F 4 "" H 6330 8495 50  0000 C CNN "Place"
-F 5 "not needed since we don't read VCC_SIM" H 6000 8840 50  0001 C CNN "Note"
+F 5 "" H 6000 8840 50  0001 C CNN "Note"
 F 6 "CRCW06031K00FKEAC" H 6000 8840 50  0001 C CNN "manf#"
 	1    6000 8840
@@
 F 3 "" H 4980 8885 60  0001 C CNN
 F 4 "" H 5310 8540 50  0000 C CNN "Place"
-F 5 "not needed since we don't read VCC_SIM" H 4980 8885 50  0001 C CNN "Note"
+F 5 "" H 4980 8885 50  0001 C CNN "Note"
 F 6 "CRCW06032K00FKEAC" H 4980 8885 50  0001 C CNN "manf#"
 	1    4980 8885
@@
 F 3 "" H 1195 8625 60  0001 C CNN
 F 4 "" H 1525 8280 50  0000 C CNN "Place"
-F 5 "not needed since we don't read VCC_SIM" H 1195 8625 50  0001 C CNN "Note"
+F 5 "" H 1195 8625 50  0001 C CNN "Note"
 F 6 "CRCW0603100KFKEAC" H 1195 8625 50  0001 C CNN "manf#"
 	1    1195 8625
@@
 	1    0    0    -1
 $EndComp
+Text Label 4660 2295 0    50   ~ 0
+RX
+Text Label 4660 2195 0    50   ~ 0
+TX
+$Comp
+L power:GND #PWR0101
+U 1 1 604667F3
+P 975 4305
+F 0 "#PWR0101" H 975 4055 50  0001 C CNN
+F 1 "GND" H 980 4132 50  0000 C CNN
+F 2 "" H 975 4305 50  0001 C CNN
+F 3 "" H 975 4305 50  0001 C CNN
+	1    975  4305
+	1    0    0    -1
+$EndComp
+Wire Wire Line
+	975  4305 975  4255
+$Comp
+L power:GND #PWR0102
+U 1 1 60475A7D
+P 1475 4330
+F 0 "#PWR0102" H 1475 4080 50  0001 C CNN
+F 1 "GND" H 1480 4157 50  0000 C CNN
+F 2 "" H 1475 4330 50  0001 C CNN
+F 3 "" H 1475 4330 50  0001 C CNN
+	1    1475 4330
+	1    0    0    -1
+$EndComp
+Wire Wire Line
+	1475 4330 1475 4280
+Wire Wire Line
+	975  3930 1060 3930
+Wire Wire Line
+	975  3930 975  4055
+Wire Wire Line
+	1475 3795 1800 3795
+Wire Wire Line
+	2050 3595 975  3595
+Wire Wire Line
+	975  3595 975  3930
+Connection ~ 975  3930
+$Comp
+L power:GND #PWR0103
+U 1 1 60512685
+P 1210 4315
+F 0 "#PWR0103" H 1210 4065 50  0001 C CNN
+F 1 "GND" H 1215 4142 50  0000 C CNN
+F 2 "" H 1210 4315 50  0001 C CNN
+F 3 "" H 1210 4315 50  0001 C CNN
+	1    1210 4315
+	1    0    0    -1
+$EndComp
+Wire Wire Line
+	1210 4315 1210 4130
+$Comp
+L Device:Crystal_GND2 Y2
+U 1 1 605379E4
+P 1210 3930
+F 0 "Y2" H 1210 4198 50  0000 C CNN
+F 1 "12Mhz" H 1210 4107 50  0000 C CNN
+F 2 "Crystal:Crystal_SMD_2520-4Pin_2.5x2.0mm" H 1210 3930 50  0001 C CNN
+F 3 "https://lcsc.com/product-detail/SMD-Crystal-Resonators_JWT-CM4012M00020T8188026_C709001.html" H 1210 3930 50  0001 C CNN
+F 4 "C709001" H 1210 3930 50  0001 C CNN "manf#"
+	1    1210 3930
+	1    0    0    -1
+$EndComp
+Wire Wire Line
+	1475 3795 1475 3930
+Wire Wire Line
+	1360 3930 1475 3930
+Connection ~ 1475 3930
+Wire Wire Line
+	1475 3930 1475 4080
 $EndSCHEMATC

Commit message: Add_BOM
Parts:
- AE1: LCSC# (none) -> C88373; manf# (none) -> U.FL-R-SMT-1(10)
- C1, C2: LCSC# (none) -> C482483; manf# (none) -> HGC0402G0220J500NTEJ
- C10, C11, C12, C13, C14, C15, C18, C19, C4, C6, C9: LCSC# (none) -> C106209; manf# (none) -> CC0402ZRY5V7BB104
- C16, C17: LCSC# (none) -> C15525; manf# TCSOM1A106M8R-ZM1 -> CL05A106MQ5NUNC
- C3, C7: LCSC# (none) -> C15684; manf# (none) -> GRM155R60J105KE19D
- C5: LCSC# (none) -> C307423; manf# CL10A475KA8NQNC -> CL05A475MQ5NRNC
- C8: LCSC# (none) -> C15684; manf# CL10A105KA8NNNC -> GRM155R60J105KE19D
- D1: LCSC# (none) -> C223608; manf# NRVB120VLSFT1G -> MBR120VLSFT1G
- D2: LCSC# (none) -> C205443; manf# 150080GS75000 -> ORH-G36G
- D3: LCSC# (none) -> C118330; manf# (none) -> D-060306R1/SS2/L
- J1: manf# AR0165 -> (none)
- P1: LCSC# (none) -> C393939; manf# (none) -> TYPE-C16PIN
- Q1: LCSC# (none) -> C96616; manf# (none) -> DMG3415U-7
- R1: LCSC# (none) -> C15458; manf# CRCW0603100KFKEAC -> 0603WAJ0104T5E
- R10, R3, R8: LCSC# (none) -> C140214; manf# (none) -> RC-02W103JT
- R11, R12: LCSC# (none) -> C131715; manf# (none) -> RK73B1JTTD512J
- R2, R9: LCSC# (none) -> C384390; manf# (none) -> WR04X102JTL
- R4, R5: LCSC# (none) -> C384351; manf# (none) -> WR04X270JTL
- R6: LCSC# (none) -> C25590; manf# CRCW06032K00FKEAC -> 0603WAJ0202T5E
- R7: LCSC# (none) -> C384390; manf# CRCW06031K00FKEAC -> WR04X102JTL
- SW1, SW2: LCSC# (none) -> C455281; manf# (none) -> TS-1088R-02526
- U1: LCSC# (none) -> C51118; manf# (none) -> AP2112K-3.3TRG1
- U3: LCSC# (none) -> C424093
- U4: LCSC# (none) -> 454-W25Q16JVUXIQTR
- Y2: LCSC# (none) -> C709001; manf# C709001 -> CM4012M00020T8188026
