File: Hardware/PicoWAN.sch (KiCad schematic (older format))
At the start: 49 parts, among them J1 Battery, J2 SWD, J3 Conn_left, J4 Conn_right, P1 USB_C_Plug_USB2.0, Q1 DMG3415U-7, SW1 BOOT, SW2 RESET, U1 AP2112K-3.3, U2 RP2040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

Commit message: nRouteinProgress
Parts:
- SW1, SW2: footprint Button_Switch_SMD:SW_SPST_TL3342 -> KiCadLibraries:TS1088R02026
Changed lines of the file:
@@
 F 0 "SW1" H 6715 5650 50  0000 C CNN
 F 1 "BOOT" H 6715 5559 50  0000 C CNN
-F 2 "Button_Switch_SMD:SW_SPST_TL3342" H 6715 5565 50  0001 C CNN
+F 2 "KiCadLibraries:TS1088R02026" H 6715 5565 50  0001 C CNN
 F 3 "https://lcsc.com/product-detail/Tactile-Switches_XUNPU-TS-1088R-02526_C455281.html" H 6715 5565 50  0001 C CNN
 F 4 "C455281" H 6715 5365 50  0001 C CNN "LCSC#"
@@
 F 0 "SW2" H 6730 6500 50  0000 C CNN
 F 1 "RESET" H 6730 6409 50  0000 C CNN
-F 2 "Button_Switch_SMD:SW_SPST_TL3342" H 6730 6415 50  0001 C CNN
+F 2 "KiCadLibraries:TS1088R02026" H 6730 6415 50  0001 C CNN
 F 3 "https://lcsc.com/product-detail/Tactile-Switches_XUNPU-TS-1088R-02526_C455281.html" H 6730 6415 50  0001 C CNN
 F 4 "C455281" H 6730 6215 50  0001 C CNN "LCSC#"

Commit message: RoutedPCB
Connections:
- net CIPO_0: now also J3.11 (Pin_11); no longer J3.13 (Pin_13)
- net COPI_0: now also J3.13 (Pin_13); no longer J3.12 (Pin_12)
- net SCK_0: now also J3.12 (Pin_12); no longer J3.11 (Pin_11)
Changed lines of the file:
@@
 Text Label 12915 2975 0    50   ~ 0
 RX
+Text Label 12915 2675 2    50   ~ 0
+CIPO_0
 Text Label 12915 2875 2    50   ~ 0
-CIPO_0
+COPI_0
 Text Label 12915 2775 2    50   ~ 0
-COPI_0
-Text Label 12915 2675 2    50   ~ 0
 SCK_0
 Text Label 14110 2770 0    50   ~ 0

Commit message: Correction_Tracks
Connections:
- net RD-: now reaches R5.2, U2.46 (USB_DM)
- net RD+: now reaches R4.2, U2.47 (USB_DP)
Changed lines of the file:
@@
 $EndComp
 Wire Wire Line
-	4550 1795 4650 1795
-Wire Wire Line
-	4550 1895 4650 1895
+	4550 1795 4605 1795
+Wire Wire Line
+	4550 1895 4605 1895
 Text Label 4950 1895 0    50   ~ 0
 D-
@@
 	1    0    0    -1
 $EndComp
+Text Label 4605 1705 1    50   ~ 0
+RD+
+Text Label 4605 1930 3    50   ~ 0
+RD-
+Wire Wire Line
+	4605 1705 4605 1795
+Connection ~ 4605 1795
+Wire Wire Line
+	4605 1795 4650 1795
+Wire Wire Line
+	4605 1930 4605 1895
+Connection ~ 4605 1895
+Wire Wire Line
+	4605 1895 4650 1895
 $EndSCHEMATC
