File: Hardware/PicoWAN.kicad_pcb (KiCad board)
At the start: 2 copper layers, 50.8 x 22.9 mm, 54 parts, among them J1 Battery, J2 SWD, J3 Conn_left, J4 Conn_right, P1 USB_C_Plug_USB2.0, Q1 DMG3415U-7, SW1 BOOT, SW2 RESET, U1 AP2112K-3.3, U2 RP2040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

Commit message: Init_rout
Parts:
- C1, C2: footprint Capacitor_SMD:C_0603_1608Metric -> Capacitor_SMD:C_0402_1005Metric
- J2: moved to B.Cu
- R2: footprint Resistor_SMD:R_0603_1608Metric_Pad1.05x0.95mm_HandSolder -> Resistor_SMD:R_0402_1005Metric
- SW1, SW2: footprint Button_Switch_SMD:SW_SPST_TL3342 -> Connectors:C455281
- moved SW2 55.2 mm to (138.4, 95.7)
- moved SW1 51.7 mm to (144.2, 95.8)
- moved C2 15.3 mm to (154.6, 89.5), turned to 135 degrees
- moved R8 12.0 mm to (170.4, 93.6), turned to 270 degrees
- moved C19 11.5 mm to (168.4, 98.2), turned to 225 degrees
- moved Y1 11.5 mm to (156.6, 88.3), turned to 225 degrees
- moved C9 11.5 mm to (161.2, 99.8), turned to 315 degrees
- moved U4 10.5 mm to (168.5, 95.6), turned to 225 degrees
- moved C7 9.66 mm to (168.7, 90.8)
- moved C4 9.27 mm to (162.0, 99.1), turned to 315 degrees
- moved R5 8.93 mm to (163.8, 98.2)
- moved R4 8.87 mm to (164.5, 98.9)
- moved C10 8.64 mm to (157.3, 95.3), turned to 225 degrees
- moved C1 8.52 mm to (157.8, 86.4), turned to 135 degrees
- moved C6 8.35 mm to (165.4, 97.2), turned to 315 degrees
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Routing:
- net +3V3: track 1.62 -> 32.3 mm
- net /D4: track 0.00 -> 24.8 mm, vias 0 -> 1
- net /RX: track 0.00 -> 23.3 mm
- net /TX: track 0.00 -> 22.7 mm, vias 0 -> 1
- net /A0: track 0.00 -> 21.9 mm, vias 0 -> 1
- net /A1: track 0.00 -> 19.5 mm, vias 0 -> 1
- net /RF_RST: track 0.00 -> 18.6 mm, vias 0 -> 1
- net /D13: track 0.00 -> 18.2 mm
- net /A2: track 0.00 -> 16.4 mm, vias 0 -> 1
- net /CIPO_0: track 0.00 -> 15.6 mm, vias 0 -> 1
- net /COPI_0: track 0.00 -> 15.2 mm, vias 0 -> 1
- net /DIO2: track 0.00 -> 15.0 mm, vias 0 -> 1
- net +BATT: track 4.53 -> 19.4 mm, vias 0 -> 1
- net /A3: track 0.00 -> 14.7 mm, vias 0 -> 1
- net /SCK_0: track 0.00 -> 14.3 mm, vias 0 -> 1
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
Commit message: Last_Change
Parts:
- moved C11 0.52 mm to (157.3, 89.8)
- moved C3 0.52 mm to (156.0, 91.1)
- moved R2 0.52 mm to (158.7, 88.4)
- moved Y1 0.52 mm to (156.2, 88.0)
- moved C1 0.52 mm to (157.4, 86.1)
- moved C2 0.52 mm to (154.2, 89.2)
Routing:
- net /SWDIO: track 0.00 -> 12.6 mm, vias 0 -> 1
- net /SWCLK: track 0.00 -> 10.1 mm, vias 0 -> 1
- net +3V3: track 32.3 -> 39.3 mm
- net GND: track 16.9 -> 23.5 mm
- net /D12: track 11.1 -> 10.4 mm
- net /D13: track 18.2 -> 17.5 mm
- net /SCK_1: track 13.0 -> 13.6 mm
- net Net-(C1-Pad1): track 6.25 -> 6.82 mm
- net +1V2: track 9.10 -> 9.62 mm

Commit message: Route
Parts:
- moved R1 2.73 mm to (136.7, 95.0), turned to 90 degrees
- moved D2 1.54 mm to (148.1, 86.7)
- moved C17 0.87 mm to (146.2, 89.0)
- moved C1 0.70 mm to (156.8, 85.8)
- moved C2 0.70 mm to (153.6, 88.9)
- moved Y1 0.70 mm to (155.6, 87.8)
- moved Q1 0.66 mm to (139.2, 92.4)
- moved R11 0.66 mm to (136.0, 91.9)
- moved D1 0.66 mm to (139.7, 95.3)
- moved J1 0.64 mm to (137.6, 88.6)
- moved R2 0.53 mm to (158.3, 88.0)
- moved C6 0.43 mm to (165.8, 96.9)
- moved C10 0.28 mm to (157.4, 95.5)
- moved C15 0.25 mm to (158.1, 96.2)
- moved C3 0.19 mm to (156.1, 91.2)
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- renumbered SW1 to BOOT, SW2 to RST
Routing:
- net +3V3: track 39.3 -> 143.7 mm, vias 0 -> 9
- net GND: track 23.5 -> 120.9 mm, vias 0 -> 17
- net /QSPI_CS: track 6.13 -> 37.6 mm, vias 0 -> 2
- net /RST: track 9.72 -> 40.3 mm, vias 1 -> 3
- net /EN: track 2.78 -> 16.0 mm, vias 0 -> 1
- net +1V2: track 9.62 -> 22.2 mm
- net /DIO5: track 13.3 -> 19.6 mm
- net /SWDIO: track 12.6 -> 9.08 mm
- net /COPI_0: track 15.1 -> 18.1 mm
- net /SWCLK: track 10.1 -> 12.7 mm
- net Net-(D2-Pad2): track 1.78 -> 3.79 mm
- net /RF_RST: track 18.7 -> 16.7 mm
- net /DIO2: track 15.0 -> 16.9 mm
- net /A0: track 21.9 -> 20.1 mm
- net Net-(R9-Pad2): track 0.00 -> 1.49 mm
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